File: dock/Main.kicad_sch (KiCad schematic)
At the start: 67 parts, among them IC401 TLV70218_SOT23-5, IC402 USBLC6-2P6, IC403 FT230XQ, IC404 MIC5219-3.3YM5, IC405 TXB0304RUT, IC406 USBLC6-2P6, IC407 USB2512BT, IC408 USBLC6-2P6, IC409 MIC2026-1xM, J401 Jumper, J402 Voltage, Q401 BSH205G2AR, SW401 Charge, X401 Debug, X402 UART, X403 Host, X404 Device, X405 Current, Y401 24 MHz

Commit message: Prepare release
- Set variant to CHECKED
- Remove unused files
- Fix ERC errors
- Fix DRC errors
- Remove Power Sequencing page
- Add block diagram

Signed-off-by: Daniel Kampert <DanielKampert@kampis-elektroecke.de>
Other:
- company: github.com/ZSWatch/Dock-HW -> ${COMPANY}
- moved on the sheet: C402, D404, R421, SW401A
